Commit message: 完成b1、b2任务

File: src/corn_robot/urdf/corn_robot.urdf (robot description, URDF)
Before this commit: robot mobile-robot, 8 links, 7 joints
Joints:
- joint base_to_lidar: origin xyz=0.2 0 0.12 rpy=0 0 -1.6 -> xyz=0.2 0 0.12 rpy=0 0 -1.65

Commit message: 完成b3\b4\b5\b6任务

File: src/corn_robot/urdf/corn_robot.urdf (robot description, URDF)
Before this commit: robot mobile-robot, 8 links, 7 joints
Joints:
- joint base_to_lidar: origin xyz=0.2 0 0.12 rpy=0 0 -1.65 -> xyz=0.2 0 0.12 rpy=0 0 -1.62

Commit message: 调优B任务

File: src/corn_robot/urdf/corn_robot.urdf (robot description, URDF)
Before this commit: robot mobile-robot, 8 links, 7 joints
Joints:
- joint base_to_lidar: origin xyz=0.2 0 0.12 rpy=0 0 -1.57 -> xyz=0.2 0 0.12 rpy=0 0 -1.6

Commit message: 修改c、d、e任务

File: src/corn_robot/urdf/corn_robot.urdf (robot description, URDF)
Before this commit: robot mobile-robot, 8 links, 7 joints
Joints:
- joint base_to_lidar: origin xyz=0.2 0 0.12 rpy=0 0 -1.6 -> xyz=0.2 0 0.12 rpy=0 0 -1.55

Commit message: 针对低矮树，调低激光雷达物理位置

File: src/corn_robot/urdf/corn_robot.urdf (robot description, URDF)
Before this commit: robot mobile-robot, 8 links, 7 joints
Links:
- removed link laser_frame
Joints:
- removed joint base_to_lidar
